File: hardware/main-board/nuBoard.kicad_pcb (KiCad board)
At the start: 6 copper layers, 141.7 x 105.1 mm, 386 parts, among them J1 FPGA Debug, J2 Barrel_Jack_Switch, J3 USB_C_Receptacle_USB2.0_16P, J4 MCU Debug, J5 Conn_01x34_Socket, J6 Conn_01x34_Socket, J7 Conn_01x34_Socket, J8 Conn_01x34_Socket, Q1 NVF5P03T3G, Q2 BSR802NL6327, SW1 MCU_Reset, SW2 MCU_Boot, U1 T120F484, U10 W25Q128JVS, U11 RP2040, U12 74LVC1G139, U13 74LVC1G139, U14 74LVC1G139, U15 74LVC1G139, U16 74LVC1G139, U17 74LVC1G139, U18 74LVC1G139, U19 74LVC1G139, U2 APS1604M-3SQRx-ZR, U20 74LVC1G139, U21 74LVC1G139, U22 74LVC1G139, U23 74LVC1G139, U24 SN74LVCH8T245PWR, U25 SN74LVCH8T245PWR, U26 SN74LVCH8T245PWR, U27 SN74LVCH8T245PWR, U28 SN74LVCH8T245PWR, U29 SN74LVCH8T245PWR, U3 TPS2116DRL, U30 SN74LVCH8T245PWR, U31 SN74LVCH8T245PWR, U32 SN74LVCH8T245PWR, U33 SN74LVCH8T245PWR, U34 SN74LVCH8T245PWR, U35 SN74LVCH8T245PWR, U36 TXS0108EPW, U37 SN74LVC1T45DRL, U38 SN74LVC1T45DRL, U39 SN74LVC1T45DRL, U4 AP2112K-3.3, U40 SN74LVC1T45DRL, U5 AP2112K-3.3, U6 TPS563201, U7 TPS563201, U8 UCC27524D, U9 TPS2111APWR, Y1 50Mhz, Y2 12Mhz

Commit message: Integrate matched top-layer HyperRAM layout and pin assignments
Parts:
- removed C135, C136, C137, C138, C139, C140, C141, C142, C143, C144: 0.1u, Capacitor_SMD:C_0201_0603Metric
- removed D10, D12, D14, D16, D18, D20, D22, D24, D26, D28, D6, D8: GREEN, LED_SMD:LED_0201_0603Metric
- removed D11, D13, D15, D17, D19, D21, D23, D25, D27, D5, D7, D9: RED, LED_SMD:LED_0201_0603Metric
- removed R44, R45, R46, R47, R48, R49, R50, R51, R52, R53, R54, R55: 1K, Resistor_SMD:R_0201_0603Metric
- removed U12, U13, U14, U15, U16, U17, U18, U19, U20, U21, U22, U23: 74LVC1G139, Package_SO:VSSOP-8_2.3x2mm_P0.5mm
- added C191: 0.1u, Capacitor_SMD:C_0402_1005Metric, B.Cu at (91.3, 76.4)
- added C192: 0.1u, Capacitor_SMD:C_0402_1005Metric, B.Cu at (90.4, 74.6)
- added R77: 10K, Resistor_SMD:R_0402_1005Metric, F.Cu at (91.7, 70.6)
- added R78: 10K, Resistor_SMD:R_0402_1005Metric, F.Cu at (89.3, 70.7)
- C133, C134: value 0.1u -> 0.01u; footprint Capacitor_SMD:C_0201_0603Metric -> Capacitor_SMD:C_0402_1005Metric
- C3: moved to B.Cu
- C4: value 1u -> 0.01u; moved to B.Cu
- U2: value APS1604M-3SQRx-ZR -> IS66WVH8M8BLL-100B1LI; footprint Package_SON:Winbond_USON-8-1EP_3x2mm_P0.5mm_EP0.2x1.6mm -> nuBoard:ISSI_TFBGA-24_6x8mm_P1.0mm
- moved U2 32.1 mm to (90.8, 75.0)
- moved C133 30.7 mm to (92.2, 73.5), turned to 90 degrees
- moved C4 30.3 mm to (91.6, 77.6), turned to 180 degrees
- moved C3 29.1 mm to (93.4, 73.5), turned to 90 degrees
- moved R13 15.7 mm to (101.6, 56.9)
- moved R14 15.7 mm to (101.6, 57.9)
- moved R15 15.7 mm to (101.6, 55.9)
- moved C134 13.8 mm to (89.2, 74.0)
- moved J2 12.4 mm to (32.1, 56.4), turned to -90 degrees
- moved C87 7.72 mm to (90.8, 81.4)
Connections:
- net /R_RCLK_EN renamed /F_RCLK_EN
- U1 pad AA16: /~{PSRAM_CE} -> unconnected-(U1F-GPIOB_RXP20-PadAA16)
- U1 pad AB16: /PSRAM_SO -> unconnected-(U1F-GPIOB_RXP28_EXTFB2-PadAB16)
- U1 pad AB17: /PSRAM_SIO2 -> unconnected-(U1F-GPIOB_RXN28_EXTFB2-PadAB17)
- U1 pad E19: /PSRAM_SIO3 -> unconnected-(U1D-GPIOR_170_CTRL15-PadE19)
- U1 pad E21: /PSRAM_SCLK -> unconnected-(U1D-GPIOR_181_CLK8-PadE21)
- U1 pad E22: /PSRAM_SI -> unconnected-(U1D-GPIOR_185_CTRL8-PadE22)
- U1 pad E5: unconnected-(U1B-GPIOL_162_EXTFB-PadE5) -> /DUT_ISOLATE
- U1 pad G1: /F_LCLK_EN -> /HR_DQ4
- U1 pad G2: /F_LCLK -> /HR_RESET_N
- U1 pad G3: /DUT_ISOLATE -> /HR_CS_N
- U1 pad G4: unconnected-(U1B-GPIOL_138-PadG4) -> /F_LCLK_EN
- U1 pad G5: unconnected-(U1B-GPIOL_147-PadG5) -> /F_LCLK
- U1 pad H1: /F_L11 -> /HR_DQ2
- U1 pad H3: /F_L10 -> unconnected-(U1B-GPIOL_131-PadH3)
- U1 pad H4: unconnected-(U1B-GPIOL_121-PadH4) -> /F_L11
- U1 pad H6: unconnected-(U1B-GPIOL_123-PadH6) -> /F_L10
- U1 pad J1: /F_L14 -> /HR_DQ3
- U1 pad J2: /F_L13 -> unconnected-(U1B-GPIOL_117-PadJ2)
- U1 pad J3: /F_L12 -> unconnected-(U1B-GPIOL_91-PadJ3)
- U1 pad J4: unconnected-(U1B-GPIOL_88-PadJ4) -> /F_L14
- U1 pad J5: unconnected-(U1B-GPIOL_85-PadJ5) -> /F_L13
- U1 pad J7: unconnected-(U1B-GPIOL_115-PadJ7) -> /F_L12
- U1 pad K1: /F_L16 -> /HR_DQ0
- U1 pad K2: /F_L15 -> /HR_DQ5
- U1 pad K4: unconnected-(U1B-GPIOL_79-PadK4) -> /F_L16
- U1 pad K5: unconnected-(U1B-GPIOL_81-PadK5) -> /F_L15
- U1 pad L1: /~{F_L1_OE} -> /HR_DQ1
- U1 pad L2: /F_L1_DIR -> /HR_DQ6
- U1 pad L3: /F_L17 -> /HR_RWDS
- U1 pad L4: unconnected-(U1B-GPIOL_74_CTRL4-PadL4) -> /~{F_L1_OE}
- U1 pad L5: unconnected-(U1B-GPIOL_71_CLK5-PadL5) -> /F_L1_DIR
- U1 pad L6: unconnected-(U1B-GPIOL_72_CLK6-PadL6) -> /F_L17
- U1 pad M1: /F_L20 -> /HR_CK
- U1 pad M3: /F_L21 -> /HR_DQ7
- U1 pad M4: unconnected-(U1B-GPIOL_64_CTRL2-PadM4) -> /F_L21
- U1 pad N4: unconnected-(U1B-GPIOL_56-PadN4) -> /F_L20
Routing:
- net +3.3V: track 221.7 -> 187.1 mm, vias 99 -> 78
- net /HR_CS_N: track 0.00 -> 18.9 mm, vias 0 -> 4
- net Net-(U1B-GPIOL_156_CBSEL0): track 7.45 -> 26.1 mm
- net Net-(U1B-GPIOL_151_TEST_N): track 2.80 -> 21.0 mm
- net /PSRAM_SO: track 17.9 -> 0.00 mm
- net GND: track 288.4 -> 272.2 mm, vias 280 -> 259
- net /HR_RESET_N: track 0.00 -> 16.0 mm
- net /FPGA_TDO: track 123.2 -> 138.8 mm, vias 5 -> 4
- net /PSRAM_SIO3: track 14.3 -> 0.00 mm, vias 2 -> 0
- net /F_L1_DIR: track 44.7 -> 31.6 mm, vias 5 -> 3
- net /PSRAM_SI: track 12.9 -> 0.00 mm
- net /PSRAM_SCLK: track 12.5 -> 0.00 mm
- net Net-(U1B-GPIOL_157_CBSEL1): track 9.21 -> 21.0 mm, vias 2 -> 3
- net /FPGA_CBUS0: track 69.1 -> 80.8 mm, vias 4 -> 9
- net /HR_RWDS: track 0.00 -> 11.2 mm
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