File: hardware/main-board/nuBoard.kicad_pcb (KiCad board)
At the start: 6 copper layers, 141.7 x 105.1 mm, 332 parts, among them J1 FPGA Debug, J2 Barrel_Jack_Switch, J3 USB_C_Receptacle_USB2.0_16P, J4 MCU Debug, J5 Conn_01x34_Socket, J6 Conn_01x34_Socket, J7 Conn_01x34_Socket, J8 Conn_01x34_Socket, Q1 NVF5P03T3G, Q2 BSR802NL6327, SW1 MCU_Reset, SW2 MCU_Boot, U1 T120F484, U10 W25Q128JVS, U11 RP2040, U2 IS66WVH8M8BLL-100B1LI, U24 SN74LVCH8T245PWR, U25 SN74LVCH8T245PWR, U26 SN74LVCH8T245PWR, U27 SN74LVCH8T245PWR, U28 SN74LVCH8T245PWR, U29 SN74LVCH8T245PWR, U3 TPS2116DRL, U30 SN74LVCH8T245PWR, U31 SN74LVCH8T245PWR, U32 SN74LVCH8T245PWR, U33 SN74LVCH8T245PWR, U34 SN74LVCH8T245PWR, U35 SN74LVCH8T245PWR, U36 TXS0108EPW, U37 SN74LVC1T45DRL, U38 SN74LVC1T45DRL, U39 SN74LVC1T45DRL, U4 AP2112K-3.3, U40 SN74LVC1T45DRL, U5 AP2112K-3.3, U6 TPS563201, U7 TPS563201, U8 UCC27524D, U9 TPS2111APWR, Y1 50Mhz, Y2 12Mhz

Commit message: Update mainboard to revision 2
Add an additional 8 bidirectional channels
Replace SPI PSRAM with hyperram
Remove LEDs
Parts:
- added C193: 0.1u, Capacitor_SMD:C_0402_1005Metric, B.Cu at (77.0, 53.7)
- added C194: 0.1u, Capacitor_SMD:C_0402_1005Metric, B.Cu at (67.0, 53.7)
- added H10: MountingHole_Pad, MountingHole:MountingHole_3.2mm_M3, F.Cu at (67.5, 113.9)
- added H11: MountingHole_Pad, MountingHole:MountingHole_3.2mm_M3, F.Cu at (100.5, 53.0)
- added H12: MountingHole_Pad, MountingHole:MountingHole_3.2mm_M3, F.Cu at (128.4, 75.8)
- added H13: MountingHole_Pad, MountingHole:MountingHole_3.2mm_M3, F.Cu at (98.0, 93.6)
- added H7: MountingHole_Pad, MountingHole:MountingHole_3.2mm_M3, F.Cu at (67.5, 39.0)
- added H8: MountingHole_Pad, MountingHole:MountingHole_3.2mm_M3, F.Cu at (148.8, 39.0)
- added H9: MountingHole_Pad, MountingHole:MountingHole_3.2mm_M3, F.Cu at (148.8, 113.9)
- added R79: 10K, Resistor_SMD:R_0402_1005Metric, B.Cu at (77.5, 56.0)
- added U41: TXS0108EPW, Package_SO:TSSOP-20_4.4x6.5mm_P0.65mm, B.Cu at (72.0, 56.0)
- H1, H2, H3, H4, H5, H6: footprint MountingHole:MountingHole_2.2mm_M2_DIN965_Pad -> MountingHole:MountingHole_3.2mm_M3_ISO7380
- U24, U25, U26, U27, U28, U29, U30, U31, U32, U33, U34, U35: value SN74LVCH8T245PWR -> SN74LVC8T245PWR
Connections:
- net /BY renamed /BX2
- net /F_BX renamed /F_BX3
- net /F_BY renamed /F_BX2
- net /F_LX renamed /F_BX1
- net /F_LY renamed /F_BX0
- net /F_RX renamed /F_RX0
- net /F_RY renamed /F_RX1
- net /F_TX renamed /F_RX2
- net /F_TY renamed /F_RX3
- net /~{F_XY_OE} renamed /~{F_X_OE}
- J5 pad 1: unconnected-(J5-Pin_1-Pad1) -> GND
- J5 pad 22: GND -> /LX0
- J5 pad 23: /LX -> /LX1
- J5 pad 24: /LY -> /LX2
- J5 pad 25: GND -> /LX3
- J6 pad 22: GND -> /TX0
- J6 pad 23: /TX -> /TX1
- J6 pad 24: /TY -> /TX2
- J6 pad 25: GND -> /TX3
- J7 pad 22: GND -> /RX0
- J7 pad 23: /RX -> /RX1
- J7 pad 24: /RY -> /RX2
- J7 pad 25: GND -> /RX3
- J8 pad 1: unconnected-(J8-Pin_1-Pad1) -> GND
- J8 pad 22: GND -> /BX0
- J8 pad 23: /BX -> /BX1
- J8 pad 25: GND -> /BX3
- U1 pad D9: unconnected-(U1C-GPIOT_TXN21-PadD9) -> /F_LX0
- U1 pad E10: unconnected-(U1C-GPIOT_TXN24-PadE10) -> /F_LX1
- U1 pad E12: unconnected-(U1C-GPIOT_RXN09_CLKN0-PadE12) -> /F_LX2
- U1 pad E6: unconnected-(U1C-GPIOT_TXN11-PadE6) -> /F_TX0
- U1 pad E8: unconnected-(U1C-GPIOT_TXP16-PadE8) -> /F_TX3
- U1 pad F10: unconnected-(U1C-GPIOT_TXP26-PadF10) -> /F_LX3
- U1 pad F6: unconnected-(U1C-GPIOT_TXP11-PadF6) -> /F_TX1
- U1 pad P5: unconnected-(U1B-GPIOL_47-PadP5) -> /F_TX2
- U36 pad 12: /LY -> /BX0
- U36 pad 13: /LX -> /BX1
- U36 pad 15: /BX -> /BX3
- U36 pad 16: /TY -> /RX3
- U36 pad 17: /TX -> /RX2
- U36 pad 18: /RY -> /RX1
- U36 pad 20: /RX -> /RX0
Routing:
- net /TY: track 151.0 -> 0.00 mm, vias 1 -> 0
- net /TX: track 148.8 -> 0.00 mm, vias 1 -> 0
- net /LX: track 108.0 -> 0.00 mm, vias 1 -> 0
- net /LY: track 102.8 -> 0.00 mm, vias 1 -> 0
- net /RY: track 82.8 -> 0.00 mm, vias 1 -> 0
- net /RX: track 75.6 -> 0.00 mm, vias 1 -> 0
- net /RX3: track 0.00 -> 70.3 mm, vias 0 -> 1
- net /~{F_X_OE}: track 25.4 -> 91.7 mm, vias 2 -> 6
- net /RX2: track 0.00 -> 64.1 mm, vias 0 -> 2
- net /RX1: track 0.00 -> 63.4 mm, vias 0 -> 1
- net /RX0: track 0.00 -> 58.2 mm, vias 0 -> 1
- net /F_LX2: track 0.00 -> 48.9 mm, vias 0 -> 4
- net /F_LX3: track 0.00 -> 47.5 mm, vias 0 -> 5
- net /F_LX1: track 0.00 -> 47.0 mm, vias 0 -> 4
- net /TX0: track 0.00 -> 42.7 mm, vias 0 -> 2
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Other:
- board text added: "Revision 2 September/2026 @wickerwaka"
- board text removed: "Revision 1 August/2026 @wickerwaka"
