File: hardware/main-board/nuBoard.kicad_sch (KiCad schematic)
At the start: 386 parts, among them J1 FPGA Debug, J2 Barrel_Jack_Switch, J3 USB_C_Receptacle_USB2.0_16P, J4 MCU Debug, J5 Conn_01x34_Socket, J6 Conn_01x34_Socket, J7 Conn_01x34_Socket, J8 Conn_01x34_Socket, Q1 NVF5P03T3G, Q2 BSR802NL6327, SW1 MCU_Reset, SW2 MCU_Boot, U1 T120F484, U10 W25Q128JVS, U11 RP2040, U12 74LVC1G139, U13 74LVC1G139, U14 74LVC1G139, U15 74LVC1G139, U16 74LVC1G139, U17 74LVC1G139, U18 74LVC1G139, U19 74LVC1G139, U2 APS1604M-3SQRx-ZR, U20 74LVC1G139, U21 74LVC1G139, U22 74LVC1G139, U23 74LVC1G139, U24 SN74LVCH8T245PWR, U25 SN74LVCH8T245PWR, U26 SN74LVCH8T245PWR, U27 SN74LVCH8T245PWR, U28 SN74LVCH8T245PWR, U29 SN74LVCH8T245PWR, U3 TPS2116DRL, U30 SN74LVCH8T245PWR, U31 SN74LVCH8T245PWR, U32 SN74LVCH8T245PWR, U33 SN74LVCH8T245PWR, U34 SN74LVCH8T245PWR, U35 SN74LVCH8T245PWR, U36 TXS0108EPW, U37 SN74LVC1T45DRL, U38 SN74LVC1T45DRL, U39 SN74LVC1T45DRL, U4 AP2112K-3.3, U40 SN74LVC1T45DRL, U5 AP2112K-3.3, U6 TPS563201, U7 TPS563201, U8 UCC27524D, U9 TPS2111APWR, Y1 50Mhz, Y2 12Mhz

Commit message: Integrate matched top-layer HyperRAM layout and pin assignments
Parts:
- removed C135, C136, C137, C138, C139, C140, C141, C142, C143, C144: 0.1u, Capacitor_SMD:C_0201_0603Metric, symbol Device:C_Small
- removed D10, D12, D14, D16, D18, D20, D22, D24, D26, D28, D6, D8: GREEN, LED_SMD:LED_0201_0603Metric, symbol Device:LED
- removed D11, D13, D15, D17, D19, D21, D23, D25, D27, D5, D7, D9: RED, LED_SMD:LED_0201_0603Metric, symbol Device:LED
- removed R44, R45, R46, R47, R48, R49, R50, R51, R52, R53, R54, R55: 1K, Resistor_SMD:R_0201_0603Metric, symbol Device:R_Small
- removed U12, U13, U14, U15, U16, U17, U18, U19, U20, U21, U22, U23: 74LVC1G139, Package_SO:VSSOP-8_2.3x2mm_P0.5mm, symbol 74xGxx:74LVC1G139
- added C191, C192: 0.1u, Capacitor_SMD:C_0402_1005Metric, symbol Device:C_Small
- added R77, R78: 10K, Resistor_SMD:R_0402_1005Metric, symbol Device:R_Small
- C133, C134: value 0.1u -> 0.01u; footprint Capacitor_SMD:C_0201_0603Metric -> Capacitor_SMD:C_0402_1005Metric; JLCPCB Part C5142565 -> (none)
- C4: value 1u -> 0.01u; JLCPCB Part C52923 -> (none)
- U2: value APS1604M-3SQRx-ZR -> IS66WVH8M8BLL-100B1LI; footprint Package_SON:Winbond_USON-8-1EP_3x2mm_P0.5mm_EP0.2x1.6mm -> nuBoard:ISSI_TFBGA-24_6x8mm_P1.0mm; symbol Memory_RAM:APS1604M-3SQRx-ZR -> HyperRAM:IS66WVH8M8BLL-100B1LI; JLCPCB Part C22423595 -> (none)
Connections:
- net +3.3V: now also U2.B4 (VCC), U2.D1 (VCCQ), U2.E4 (VCCQ), C191.1, C192.1, R77.1, R78.1; no longer U2.8 (VDD)
- net DUT_ISOLATE: now also U1.E5 (GPIOL_162_EXTFB); no longer U1.G3 (GPIOL_141)
- net F_L10: now also U1.H6 (GPIOL_123); no longer U1.H3 (GPIOL_131)
- net F_L11: now also U1.H4 (GPIOL_121); no longer U1.H1 (GPIOL_133)
- net F_L12: now also U1.J7 (GPIOL_115); no longer U1.J3 (GPIOL_91)
- net F_L13: now also U1.J5 (GPIOL_85); no longer U1.J2 (GPIOL_117)
- net F_L14: now also U1.J4 (GPIOL_88); no longer U1.J1 (GPIOL_119)
- net F_L15: now also U1.K5 (GPIOL_81); no longer U1.K2 (GPIOL_89)
- net F_L16: now also U1.K4 (GPIOL_79); no longer U1.K1 (GPIOL_87)
- net F_L17: now also U1.L6 (GPIOL_72_CLK6); no longer U1.L3 (GPIOL_73_CLK7)
- net F_L1_DIR: now also U1.L5 (GPIOL_71_CLK5); no longer U1.L2 (GPIOL_69_CLK3)
- net F_L20: now also U1.N4 (GPIOL_56); no longer U1.M1 (GPIOL_65_CTRL3)
- net F_L21: now also U1.M4 (GPIOL_64_CTRL2); no longer U1.M3 (GPIOL_67_CLK1)
- net F_LCLK: now also U1.G5 (GPIOL_147); no longer U1.G2 (GPIOL_142)
- net F_LCLK_EN: now also U1.G4 (GPIOL_138); no longer U1.G1 (GPIOL_136)
- net GND: now also U2.B3 (VSS), U2.C1 (VSSQ), U2.E5 (VSSQ), C191.2, C192.2; no longer U2.4 (VSS), U2.9 (EPAD)
- net ~{F_L1_OE}: now also U1.L4 (GPIOL_74_CTRL4); no longer U1.L1 (GPIOL_68_CLK2)
- net PSRAM_SCLK: no longer names the net of U1.E21 (GPIOR_181_CLK8)
- net PSRAM_SCLK: no longer U2.6 (SCLK)
- net PSRAM_SI: no longer names the net of U1.E22 (GPIOR_185_CTRL8)
- net PSRAM_SI: no longer U2.5 (SI/SIO0)
- net PSRAM_SIO2: no longer names the net of U1.AB17 (GPIOB_RXN28_EXTFB2)
- net PSRAM_SIO2: no longer U2.3 (SIO2)
- net PSRAM_SIO3: no longer names the net of U1.E19 (GPIOR_170_CTRL15)
- net PSRAM_SIO3: no longer U2.7 (SIO3)
- net PSRAM_SO: no longer names the net of U1.AB16 (GPIOB_RXP28_EXTFB2)
- net PSRAM_SO: no longer U2.2 (SO/SIO1)
- net R_RCLK_EN renamed F_RCLK_EN
- net ~{PSRAM_CE}: no longer names the net of U1.AA16 (GPIOB_RXP20)
- net ~{PSRAM_CE}: no longer U2.1 (~{CE})
- new net HR_CK: U1.M1 (GPIOL_65_CTRL3), U2.B2 (CK)
- new net HR_CS_N: R77.2, U1.G3 (GPIOL_141), U2.A3 (~{CS})
- new net HR_DQ0: U1.K1 (GPIOL_87), U2.D3 (DQ0)
- new net HR_DQ1: U1.L1 (GPIOL_68_CLK2), U2.D2 (DQ1)
- new net HR_DQ2: U1.H1 (GPIOL_133), U2.C4 (DQ2)
- new net HR_DQ3: U1.J1 (GPIOL_119), U2.D4 (DQ3)
- new net HR_DQ4: U1.G1 (GPIOL_136), U2.D5 (DQ4)
- new net HR_DQ5: U1.K2 (GPIOL_89), U2.E3 (DQ5)
- new net HR_DQ6: U1.L2 (GPIOL_69_CLK3), U2.E2 (DQ6)
- new net HR_DQ7: U1.M3 (GPIOL_67_CLK1), U2.E1 (DQ7)
- new net HR_RESET_N: R78.2, U1.G2 (GPIOL_142), U2.A4 (~{RESET})
- new net HR_RWDS: U1.L3 (GPIOL_73_CLK7), U2.C3 (RWDS)
- no-connect marks 115 -> 113
Other:
- note added: "HyperRAM: F.Cu-only, no vias; CK/DQ[7:0]/RWDS verified PCB length spread 0.214807mm (limit 0.381mm). U2 and signal tracks locked. Package skew excluded; power/pull-ups and FPGA timing remain unfinished."
- note removed: "DIR"
- note removed: "~{OE}"
- moved on the sheet: C4

Commit message: Update mainboard to revision 2
Add an additional 8 bidirectional channels
Replace SPI PSRAM with hyperram
Remove LEDs
Parts:
- added C193, C194: 0.1u, Capacitor_SMD:C_0402_1005Metric, symbol Device:C_Small
- added H10, H11, H12, H13, H7, H8, H9: MountingHole_Pad, MountingHole:MountingHole_3.2mm_M3, symbol Mechanical:MountingHole
- added R79: 10K, Resistor_SMD:R_0402_1005Metric, symbol Device:R_Small
- added U41: TXS0108EPW, Package_SO:TSSOP-20_4.4x6.5mm_P0.65mm, symbol Logic_LevelTranslator:TXS0108EPW
- C133, C134, C4: JLCPCB Part (none) -> C15195
- H1, H2, H3, H4, H5, H6: footprint MountingHole:MountingHole_2.2mm_M2_DIN965_Pad -> MountingHole:MountingHole_3.2mm_M3_ISO7380; symbol Mechanical:MountingHole_Pad -> Mechanical:MountingHole
- R77, R78: JLCPCB Part (none) -> C25744
- U2: JLCPCB Part (none) -> C1349096
- U24, U25, U26, U27, U28, U29, U30, U31, U32, U33, U34, U35: value SN74LVCH8T245PWR -> SN74LVC8T245PWR; JLCPCB Part C201741 -> C27643
Connections:
- net +3.3V: now also C193.1, R79.1, U41.2 (VCCA)
- net GND: now also J5.1 (Pin_1), J8.1 (Pin_1), C193.2, C194.2, U41.11 (GND); no longer H1.1, H2.1, H3.1, H4.1, H5.1, H6.1, J5.22 (Pin_22), J5.25 (Pin_25), J6.22 (Pin_22), J6.25 (Pin_25), J7.22 (Pin_22), J7.25 (Pin_25), J8.22 (Pin_22), J8.25 (Pin_25)
- net VCCB: now also C194.1, U41.19 (VCCB)
- net F_LX0: now reaches U1.D9 (GPIOT_TXN21)
- net F_LX0: now also U41.6 (A5)
- net F_LX1: now reaches U1.E10 (GPIOT_TXN24)
- net F_LX1: now also U41.7 (A6)
- net F_LX2: now reaches U1.E12 (GPIOT_RXN09_CLKN0)
- net F_LX2: now also U41.8 (A7)
- net F_TX0: now reaches U1.E6 (GPIOT_TXN11)
- net F_TX0: now also U41.1 (A1)
- net F_TX3: now reaches U1.E8 (GPIOT_TXP16)
- net F_TX3: now also U41.5 (A4)
- net F_LX3: now reaches U1.F10 (GPIOT_TXP26)
- net F_LX3: now also U41.9 (A8)
- net F_TX1: now reaches U1.F6 (GPIOT_TXP11)
- net F_TX1: now also U41.3 (A2)
- net F_TX2: now reaches U1.P5 (GPIOL_47)
- net F_TX2: now also U41.4 (A3)
- net BX renamed BX1
- net BX1: now also U36.13 (B7); no longer U36.15 (B5)
- net BY renamed BX2
- net F_BX renamed F_BX3
- net F_BY renamed F_BX2
- net F_LX renamed F_BX1
- net F_LY renamed F_BX0
- net F_RX renamed F_RX0
- net F_RY renamed F_RX1
- net F_TX renamed F_RX2
- net F_TY renamed F_RX3
- net LX renamed LX1
- net LX1: now also U41.14 (B6); no longer U36.13 (B7)
- net LY renamed BX0
- net BX0: now also J8.22 (Pin_22); no longer J5.24 (Pin_24)
- net RX renamed RX0
- net RX0: now also J7.22 (Pin_22); no longer J7.23 (Pin_23)
- net RY renamed RX1
- net RX1: now also J7.23 (Pin_23); no longer J7.24 (Pin_24)
- net TX renamed RX2
- net RX2: now also J7.24 (Pin_24); no longer J6.23 (Pin_23)
- net TY renamed RX3
- net RX3: now also J7.25 (Pin_25); no longer J6.24 (Pin_24)
- net ~{F_XY_OE} renamed ~{F_X_OE}
- net ~{F_X_OE}: now also R79.2, U41.10 (OE)
- new net BX3: J8.25 (Pin_25), U36.15 (B5)
- new net LX0: J5.22 (Pin_22), U41.15 (B5)
- new net LX2: J5.24 (Pin_24), U41.13 (B7)
- new net LX3: J5.25 (Pin_25), U41.12 (B8)
- new net TX0: J6.22 (Pin_22), U41.20 (B1)
- new net TX1: J6.23 (Pin_23), U41.18 (B2)
- new net TX2: J6.24 (Pin_24), U41.17 (B3)
- new net TX3: J6.25 (Pin_25), U41.16 (B4)
- no-connect marks 113 -> 110
Other:
- note added: "Extraction Holes"
- note added: "HyperRAM: F.Cu-only, no vias; CK/DQ[7:0]/RWDS verified PCB length spread 0.214807mm (limit 0.381mm). U2 and signal tracks locked. Package skew excluded;"
- note added: "Mounting Holes"
- note removed: "HyperRAM: F.Cu-only, no vias; CK/DQ[7:0]/RWDS verified PCB length spread 0.214807mm (limit 0.381mm). U2 and signal tracks locked. Package skew excluded; power/pull-ups and FPGA timing remain unfinished."

Commit message: Fit power inductors for the FPGA buck converters
L1 and L2 used C16903, a ferrite bead, which made U6 and U7 whine and
damaged U6. Switch to C964122 in a 1008 footprint. Note that the
HyperRAM is held deselected until it is supported.

Claude-Session: https://claude.ai/code/session_01Mb721YdebqpSQrfvW2MyND
Parts:
- L1, L2: footprint Inductor_SMD:L_0805_2012Metric -> Inductor_SMD:L_1008_2520Metric; JLCPCB Part C16903 -> C964122
Changed lines of the file:
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@@
 			)
 		)
-		(property "Footprint" "Inductor_SMD:L_0805_2012Metric"
+		(property "Footprint" "Inductor_SMD:L_1008_2520Metric"
 			(at 593.09 111.76 0)
 			(hide yes)
@@
 			)
 		)
-		(property "JLCPCB Part" "C16903"
+		(property "JLCPCB Part" "C964122"
 			(at 593.09 111.76 90)
 			(hide yes)
@@
 			)
 		)
-		(property "Footprint" "Inductor_SMD:L_0805_2012Metric"
+		(property "Footprint" "Inductor_SMD:L_1008_2520Metric"
 			(at 593.09 154.94 0)
 			(hide yes)
@@
 			)
 		)
-		(property "JLCPCB Part" "C16903"
+		(property "JLCPCB Part" "C964122"
 			(at 593.09 154.94 90)
 			(hide yes)
