File: hardware/68000/68000.kicad_sch (KiCad schematic)
At the start: 6 parts, among them J1 nuMezzanine_4x34, U1 MC68000P

Commit message: Update mainboard to revision 2
Add an additional 8 bidirectional channels
Replace SPI PSRAM with hyperram
Remove LEDs
Parts:
- C1, C2: footprint Capacitor_THT:C_Disc_D4.7mm_W2.5mm_P5.00mm -> Capacitor_SMD:C_0805_2012Metric_Pad1.18x1.45mm_HandSolder
- R1, R2: footprint Resistor_THT:R_Axial_DIN0207_L6.3mm_D2.5mm_P7.62mm_Horizontal -> Resistor_SMD:R_0805_2012Metric_Pad1.20x1.40mm_HandSolder
Connections:
- net GND: now also J1.102 (GND), J1.136 (GND); no longer J1.10 (GND), J1.112 (GND), J1.115 (GND), J1.13 (GND), J1.44 (GND), J1.47 (GND), J1.78 (GND), J1.81 (GND)
- net BX renamed BX1
- net BY renamed BX2
- net LX renamed LX1
- net LY renamed LX2
- net RX renamed RX1
- net RY renamed RX2
- net TX renamed TX1
- net TY renamed TX2
- no-connect marks 4 -> 12
Changed lines of the file:
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@@
 		)
 	)
-	(label "TX"
+	(label "TX1"
 		(at 36.83 97.79 0)
 		(effects
@@
 		)
 	)
-	(label "LY"
+	(label "LX2"
 		(at 36.83 191.77 0)
 		(effects
@@
 		)
 	)
-	(label "BY"
+	(label "BX2"
 		(at 72.39 100.33 0)
 		(effects
@@
 		)
 	)
-	(label "RX"
+	(label "RX1"
 		(at 72.39 189.23 0)
 		(effects
@@
 		)
 	)
-	(label "LY"
+	(label "LX2"
 		(at 148.59 139.7 180)
 		(effects
@@
 		)
 	)
-	(label "LX"
+	(label "LX1"
 		(at 148.59 121.92 180)
 		(effects
@@
 		)
 	)
-	(label "BX"
+	(label "BX1"
 		(at 72.39 97.79 0)
 		(effects
@@
 		)
 	)
-	(label "TY"
+	(label "TX2"
 		(at 36.83 100.33 0)
 		(effects
@@
 		)
 	)
-	(label "RY"
+	(label "RX2"
 		(at 72.39 191.77 0)
 		(effects
@@
 		)
 	)
-	(label "LX"
+	(label "LX1"
 		(at 36.83 189.23 0)
 		(effects
@@
 			)
 		)
-		(property "Footprint" "Resistor_THT:R_Axial_DIN0207_L6.3mm_D2.5mm_P7.62mm_Horizontal"
+		(property "Footprint" "Resistor_SMD:R_0805_2012Metric_Pad1.20x1.40mm_HandSolder"
 			(at 149.352 118.11 90)
 			(hide yes)
@@
 			)
 		)
-		(property "Footprint" "Resistor_THT:R_Axial_DIN0207_L6.3mm_D2.5mm_P7.62mm_Horizontal"
+		(property "Footprint" "Resistor_SMD:R_0805_2012Metric_Pad1.20x1.40mm_HandSolder"
 			(at 159.512 135.89 90)
 			(hide yes)
@@
 			)
 		)
-		(property "Footprint" "Capacitor_THT:C_Disc_D4.7mm_W2.5mm_P5.00mm"
+		(property "Footprint" "Capacitor_SMD:C_0805_2012Metric_Pad1.18x1.45mm_HandSolder"
 			(at 211.7852 30.48 0)
 			(hide yes)
@@
 			)
 		)
-		(property "Footprint" "Capacitor_THT:C_Disc_D4.7mm_W2.5mm_P5.00mm"
+		(property "Footprint" "Capacitor_SMD:C_0805_2012Metric_Pad1.18x1.45mm_HandSolder"
 			(at 221.9452 30.48 0)
 			(hide yes)
@@
 	)
 	(embedded_fonts no)
+(no_connect (at 36.83 186.69))
+(no_connect (at 36.83 194.31))
+(no_connect (at 36.83 95.25))
+(no_connect (at 36.83 102.87))
+(no_connect (at 72.39 186.69))
+(no_connect (at 72.39 194.31))
+(no_connect (at 72.39 95.25))
+(no_connect (at 72.39 102.87))
 )
