File: hardware/68030/68030.kicad_sch (KiCad schematic)
At the start: 20 parts, among them J1 nuMezzanine_4x34, U1 MC68030RC25B

Commit message: Update mainboard to revision 2
Add an additional 8 bidirectional channels
Replace SPI PSRAM with hyperram
Remove LEDs
Parts:
- C1, C10, C11, C12, C13, C14, C15, C2, C3, C4, C5, C6, C7, C8, C9: footprint Capacitor_THT:C_Disc_D5.0mm_W2.5mm_P5.00mm -> Capacitor_SMD:C_0805_2012Metric_Pad1.18x1.45mm_HandSolder
- C16: footprint Capacitor_THT:CP_Radial_D5.0mm_P2.00mm -> Capacitor_SMD:C_0805_2012Metric_Pad1.18x1.45mm_HandSolder; symbol Device:C_Polarized -> Device:C; Dielectric aluminum electrolytic -> X7R/X5R MLCC
- R1, R2: footprint Resistor_THT:R_Axial_DIN0207_L6.3mm_D2.5mm_P7.62mm_Horizontal -> Resistor_SMD:R_0805_2012Metric_Pad1.20x1.40mm_HandSolder
Connections:
- net GND: now also J1.102 (GND), J1.136 (GND); no longer J1.10 (GND), J1.112 (GND), J1.115 (GND), J1.13 (GND), J1.44 (GND), J1.47 (GND), J1.78 (GND), J1.81 (GND)
- net BX renamed BX1
- net BY renamed BX2
- net LX renamed LX1
- net LY renamed LX2
- net RX renamed RX1
- net RY renamed RX2
- net TX renamed TX1
- net TY renamed TX2
- no-connect marks 12 -> 20
Other:
- note added: "HOST CONTRACT 5V_SELECT grounded; 3V3_SELECT floating. CPU clock: 12.5-25 MHz; timing not yet qualified. X1/X2: open-drain only; keep enabled, release HIGH, never drive HIGH. Internal host pulls used. Preload all tied unused bank bits LOW before every host-output enable. Respect byte lanes and bus-release delays; never drive always-output bank. CPU TTL output-high and host keeper margins are NOT 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"
- note removed: "HOST CONTRACT 5V_SELECT grounded; 3V3_SELECT floating. CPU clock: 12.5-25 MHz; timing not yet qualified. X/Y: open-drain only; keep enabled, release HIGH, never drive HIGH. Internal host pulls used. Preload all tied unused bank bits LOW before every host-output enable. Respect byte lanes and bus-release delays; never drive always-output bank. CPU TTL output-high and host keeper margins are NOT gu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"
Changed lines of the file:
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@@
       (type default))
 )
-  (label "LY"
+  (label "LX2"
     (at 40.64 191.77 0)
     (effects
@@
       (type default))
 )
-  (label "LX"
+  (label "LX1"
     (at 40.64 189.23 0)
     (effects
@@
       (type default))
 )
-  (label "TY"
+  (label "TX2"
     (at 40.64 100.33 0)
     (effects
@@
       (type default))
 )
-  (label "TX"
+  (label "TX1"
     (at 40.64 97.79 0)
     (effects
@@
       (type default))
 )
-  (label "RY"
+  (label "RX2"
     (at 76.2 191.77 0)
     (effects
@@
       (type default))
 )
-  (label "RX"
+  (label "RX1"
     (at 76.2 189.23 0)
     (effects
@@
       (type default))
 )
-  (label "BY"
+  (label "BX2"
     (at 76.2 100.33 0)
     (effects
@@
       (type default))
 )
-  (label "BX"
+  (label "BX1"
     (at 76.2 97.79 0)
     (effects
@@
       (type default))
 )
-  (label "TX"
+  (label "TX1"
     (at 384.81 162.56 180)
     (effects
@@
       (type default))
 )
-  (label "BY"
+  (label "BX2"
     (at 384.81 165.1 180)
     (effects
@@
       (type default))
 )
-  (label "RX"
+  (label "RX1"
     (at 384.81 167.64 180)
     (effects
@@
       (type default))
 )
-  (label "LY"
+  (label "LX2"
     (at 384.81 170.18 180)
     (effects
@@
       (type default))
 )
-  (label "BX"
+  (label "BX1"
     (at 384.81 172.72 180)
     (effects
@@
       (type default))
 )
-  (label "RY"
+  (label "RX2"
     (at 384.81 175.26 180)
     (effects
@@
       (type default))
 )
-  (label "TY"
+  (label "TX2"
     (at 384.81 177.8 180)
     (effects
@@
       (type default))
 )
-  (label "LX"
+  (label "LX1"
     (at 384.81 180.34 180)
     (effects
@@
           (size 1.27 1.27))
         (justify left)))
-    (property "Footprint" "Capacitor_THT:C_Disc_D5.0mm_W2.5mm_P5.00mm"
+    (property "Footprint" "Capacitor_SMD:C_0805_2012Metric_Pad1.18x1.45mm_HandSolder"
       (at 355.6 246.38 0)
       (effects
@@
           (size 1.27 1.27))
         (justify left)))
-    (property "Footprint" "Capacitor_THT:C_Disc_D5.0mm_W2.5mm_P5.00mm"
+    (property "Footprint" "Capacitor_SMD:C_0805_2012Metric_Pad1.18x1.45mm_HandSolder"
       (at 393.7 246.38 0)
       (effects
@@
           (size 1.27 1.27))
         (justify left)))
-    (property "Footprint" "Capacitor_THT:C_Disc_D5.0mm_W2.5mm_P5.00mm"
+    (property "Footprint" "Capacitor_SMD:C_0805_2012Metric_Pad1.18x1.45mm_HandSolder"
       (at 431.8 246.38 0)
       (effects
@@
           (size 1.27 1.27))
         (justify left)))
-    (property "Footprint" "Capacitor_THT:C_Disc_D5.0mm_W2.5mm_P5.00mm"
+    (property "Footprint" "Capacitor_SMD:C_0805_2012Metric_Pad1.18x1.45mm_HandSolder"
       (at 469.9 246.38 0)
       (effects
@@
           (size 1.27 1.27))
         (justify left)))
-    (property "Footprint" "Capacitor_THT:C_Disc_D5.0mm_W2.5mm_P5.00mm"
+    (property "Footprint" "Capacitor_SMD:C_0805_2012Metric_Pad1.18x1.45mm_HandSolder"
       (at 508.0 246.38 0)
       (effects
@@
           (size 1.27 1.27))
         (justify left)))
-    (property "Footprint" "Capacitor_THT:C_Disc_D5.0mm_W2.5mm_P5.00mm"
+    (property "Footprint" "Capacitor_SMD:C_0805_2012Metric_Pad1.18x1.45mm_HandSolder"
       (at 355.6 276.86 0)
       (effects
@@
           (size 1.27 1.27))
         (justify left)))
-    (property "Footprint" "Capacitor_THT:C_Disc_D5.0mm_W2.5mm_P5.00mm"
+    (property "Footprint" "Capacitor_SMD:C_0805_2012Metric_Pad1.18x1.45mm_HandSolder"
       (at 393.7 276.86 0)
       (effects
@@
           (size 1.27 1.27))
         (justify left)))
-    (property "Footprint" "Capacitor_THT:C_Disc_D5.0mm_W2.5mm_P5.00mm"
+    (property "Footprint" "Capacitor_SMD:C_0805_2012Metric_Pad1.18x1.45mm_HandSolder"
       (at 431.8 276.86 0)
       (effects
@@
           (size 1.27 1.27))
         (justify left)))
-    (property "Footprint" "Capacitor_THT:C_Disc_D5.0mm_W2.5mm_P5.00mm"
+    (property "Footprint" "Capacitor_SMD:C_0805_2012Metric_Pad1.18x1.45mm_HandSolder"
       (at 469.9 276.86 0)
       (effects
@@
           (size 1.27 1.27))
         (justify left)))
-    (property "Footprint" "Capacitor_THT:C_Disc_D5.0mm_W2.5mm_P5.00mm"
+    (property "Footprint" "Capacitor_SMD:C_0805_2012Metric_Pad1.18x1.45mm_HandSolder"
       (at 508.0 276.86 0)
       (effects
@@
           (size 1.27 1.27))
         (justify left)))
-    (property "Footprint" "Capacitor_THT:C_Disc_D5.0mm_W2.5mm_P5.00mm"
+    (property "Footprint" "Capacitor_SMD:C_0805_2012Metric_Pad1.18x1.45mm_HandSolder"
       (at 355.6 307.34 0)
       (effects
@@
           (size 1.27 1.27))
         (justify left)))
-    (property "Footprint" "Capacitor_THT:C_Disc_D5.0mm_W2.5mm_P5.00mm"
+    (property "Footprint" "Capacitor_SMD:C_0805_2012Metric_Pad1.18x1.45mm_HandSolder"
       (at 393.7 307.34 0)
       (effects
@@
           (size 1.27 1.27))
         (justify left)))
-    (property "Footprint" "Capacitor_THT:C_Disc_D5.0mm_W2.5mm_P5.00mm"
+    (property "Footprint" "Capacitor_SMD:C_0805_2012Metric_Pad1.18x1.45mm_HandSolder"
       (at 431.8 307.34 0)
       (effects
@@
           (size 1.27 1.27))
         (justify left)))
-    (property "Footprint" "Capacitor_THT:C_Disc_D5.0mm_W2.5mm_P5.00mm"
+    (property "Footprint" "Capacitor_SMD:C_0805_2012Metric_Pad1.18x1.45mm_HandSolder"
       (at 469.9 307.34 0)
       (effects
@@
           (size 1.27 1.27))
         (justify left)))
-    (property "Footprint" "Capacitor_THT:C_Disc_D5.0mm_W2.5mm_P5.00mm"
+    (property "Footprint" "Capacitor_SMD:C_0805_2012Metric_Pad1.18x1.45mm_HandSolder"
       (at 508.0 307.34 0)
       (effects
@@
 )
   (symbol
-    (lib_id "Device:C_Polarized")
+    (lib_id "Device:C")
     (at 355.6 342.9 0)
     (unit 1)
@@
           (size 1.27 1.27))
         (justify left)))
-    (property "Footprint" "Capacitor_THT:CP_Radial_D5.0mm_P2.00mm"
+    (property "Footprint" "Capacitor_SMD:C_0805_2012Metric_Pad1.18x1.45mm_HandSolder"
       (at 355.6 342.9 0)
       (effects
@@
           (size 1.27 1.27))
         (hide yes)))
-    (property "Dielectric" "aluminum electrolytic"
+    (property "Dielectric" "X7R/X5R MLCC"
       (at 355.6 342.9 0)
       (effects
@@
           (size 1.27 1.27))
         (justify left)))
-    (property "Footprint" "Resistor_THT:R_Axial_DIN0207_L6.3mm_D2.5mm_P7.62mm_Horizontal"
+    (property "Footprint" "Resistor_SMD:R_0805_2012Metric_Pad1.20x1.40mm_HandSolder"
       (at 165.1 337.82 0)
       (effects
@@
           (size 1.27 1.27))
         (justify left)))
-    (property "Footprint" "Resistor_THT:R_Axial_DIN0207_L6.3mm_D2.5mm_P7.62mm_Horizontal"
+    (property "Footprint" "Resistor_SMD:R_0805_2012Metric_Pad1.20x1.40mm_HandSolder"
       (at 241.3 337.82 0)
       (effects
@@
     (rev "1.0")
     (comment 1 "CPGA128 / 5 V / full bus, burst and takeover / experimental direct interface"))
-  (text "HOST CONTRACT\n5V_SELECT grounded; 3V3_SELECT floating. CPU clock: 12.5-25 MHz; timing not yet qualified.\nX/Y: open-drain only; keep enabled, release HIGH, never drive HIGH. Internal host pulls used.\nPreload all tied unused bank bits LOW before every host-output enable.\nRespect byte lanes and bus-release delays; never drive always-output bank.\nCPU TTL output-high and host keeper margins are NOT guaranteed. See design-notes.md."
+  (text "HOST CONTRACT\n5V_SELECT grounded; 3V3_SELECT floating. CPU clock: 12.5-25 MHz; timing not yet qualified.\nX1/X2: open-drain only; keep enabled, release HIGH, never drive HIGH. Internal host pulls used.\nPreload all tied unused bank bits LOW before every host-output enable.\nRespect byte lanes and bus-release delays; never drive always-output bank.\nCPU TTL output-high and host keeper margins are NOT guaranteed. See design-notes.md."
     (at 255.27 383.54 0)
     (effects
       (font
         (size 1.1 1.1)))
-))
+)(no_connect (at 36.83 186.69))
+(no_connect (at 36.83 194.31))
+(no_connect (at 36.83 95.25))
+(no_connect (at 36.83 102.87))
+(no_connect (at 72.39 186.69))
+(no_connect (at 72.39 194.31))
+(no_connect (at 72.39 95.25))
+(no_connect (at 72.39 102.87))
+)
