File: hardware/daughter-template/nuDaughter.kicad_pcb (KiCad board)
At the start: 2 copper layers, 99.1 x 99.1 mm, 1 part, among them J1 nuMezzanine_4x34

Commit message: Update mainboard to revision 2
Add an additional 8 bidirectional channels
Replace SPI PSRAM with hyperram
Remove LEDs
Connections:
- J1 pad 10: GND -> /TX3
- J1 pad 100: unconnected-(J1C-B00-Pad100) -> /B00
- J1 pad 102: unconnected-(J1E-NC-Pad102) -> GND
- J1 pad 104: unconnected-(J1B-L27-Pad104) -> /L27
- J1 pad 105: unconnected-(J1B-L26-Pad105) -> /L26
- J1 pad 106: unconnected-(J1B-L25-Pad106) -> /L25
- J1 pad 107: unconnected-(J1B-L24-Pad107) -> /L24
- J1 pad 108: unconnected-(J1B-L23-Pad108) -> /L23
- J1 pad 109: unconnected-(J1B-L22-Pad109) -> /L22
- J1 pad 11: unconnected-(J1A-TY-Pad11) -> /TX2
- J1 pad 110: unconnected-(J1B-L21-Pad110) -> /L21
- J1 pad 111: unconnected-(J1B-L20-Pad111) -> /L20
- J1 pad 112: GND -> /LX3
- J1 pad 113: unconnected-(J1B-LY-Pad113) -> /LX2
- J1 pad 114: unconnected-(J1B-LX-Pad114) -> /LX1
- J1 pad 115: GND -> /LX0
- J1 pad 116: unconnected-(J1B-L17-Pad116) -> /L17
- J1 pad 117: unconnected-(J1B-L16-Pad117) -> /L16
- J1 pad 118: unconnected-(J1B-L15-Pad118) -> /L15
- J1 pad 119: unconnected-(J1B-L14-Pad119) -> /L14
- J1 pad 12: unconnected-(J1A-TX-Pad12) -> /TX1
- J1 pad 120: unconnected-(J1B-L13-Pad120) -> /L13
- J1 pad 121: unconnected-(J1B-L12-Pad121) -> /L12
- J1 pad 122: unconnected-(J1B-L11-Pad122) -> /L11
- J1 pad 123: unconnected-(J1B-L10-Pad123) -> /L10
- J1 pad 125: unconnected-(J1B-LCLK-Pad125) -> /LCLK
- J1 pad 127: unconnected-(J1B-L07-Pad127) -> /L07
- J1 pad 128: unconnected-(J1B-L06-Pad128) -> /L06
- J1 pad 129: unconnected-(J1B-L05-Pad129) -> /L05
- J1 pad 13: GND -> /TX0
- J1 pad 130: unconnected-(J1B-L04-Pad130) -> /L04
- J1 pad 131: unconnected-(J1B-L03-Pad131) -> /L03
- J1 pad 132: unconnected-(J1B-L02-Pad132) -> /L02
- J1 pad 133: unconnected-(J1B-L01-Pad133) -> /L01
- J1 pad 134: unconnected-(J1B-L00-Pad134) -> /L00
- J1 pad 136: unconnected-(J1E-NC-Pad136) -> GND
- J1 pad 14: unconnected-(J1A-T17-Pad14) -> /T17
- J1 pad 15: unconnected-(J1A-T16-Pad15) -> /T16
- J1 pad 16: unconnected-(J1A-T15-Pad16) -> /T15
- J1 pad 17: unconnected-(J1A-T14-Pad17) -> /T14
- J1 pad 18: unconnected-(J1A-T13-Pad18) -> /T13
- J1 pad 19: unconnected-(J1A-T12-Pad19) -> /T12
- J1 pad 2: unconnected-(J1A-T27-Pad2) -> /T27
- J1 pad 20: unconnected-(J1A-T11-Pad20) -> /T11
- J1 pad 21: unconnected-(J1A-T10-Pad21) -> /T10
- J1 pad 23: unconnected-(J1A-TCLK-Pad23) -> /TCLK
- J1 pad 25: unconnected-(J1A-T07-Pad25) -> /T07
- J1 pad 26: unconnected-(J1A-T06-Pad26) -> /T06
- J1 pad 27: unconnected-(J1A-T05-Pad27) -> /T05
- J1 pad 28: unconnected-(J1A-T04-Pad28) -> /T04
- J1 pad 29: unconnected-(J1A-T03-Pad29) -> /T03
- J1 pad 3: unconnected-(J1A-T26-Pad3) -> /T26
- J1 pad 30: unconnected-(J1A-T02-Pad30) -> /T02
- J1 pad 31: unconnected-(J1A-T01-Pad31) -> /T01
- J1 pad 32: unconnected-(J1A-T00-Pad32) -> /T00
- J1 pad 36: unconnected-(J1D-R27-Pad36) -> /R27
- J1 pad 37: unconnected-(J1D-R26-Pad37) -> /R26
- J1 pad 38: unconnected-(J1D-R25-Pad38) -> /R25
- J1 pad 39: unconnected-(J1D-R24-Pad39) -> /R24
- J1 pad 4: unconnected-(J1A-T25-Pad4) -> /T25
- J1 pad 40: unconnected-(J1D-R23-Pad40) -> /R23
- J1 pad 41: unconnected-(J1D-R22-Pad41) -> /R22
- J1 pad 42: unconnected-(J1D-R21-Pad42) -> /R21
- J1 pad 43: unconnected-(J1D-R20-Pad43) -> /R20
- J1 pad 44: GND -> /RX3
- J1 pad 45: unconnected-(J1D-RY-Pad45) -> /RX2
- J1 pad 46: unconnected-(J1D-RX-Pad46) -> /RX1
- J1 pad 47: GND -> /RX0
- J1 pad 48: unconnected-(J1D-R17-Pad48) -> /R17
- J1 pad 49: unconnected-(J1D-R16-Pad49) -> /R16
- J1 pad 5: unconnected-(J1A-T24-Pad5) -> /T24
- J1 pad 50: unconnected-(J1D-R15-Pad50) -> /R15
- J1 pad 51: unconnected-(J1D-R14-Pad51) -> /R14
- J1 pad 52: unconnected-(J1D-R13-Pad52) -> /R13
- J1 pad 53: unconnected-(J1D-R12-Pad53) -> /R12
- J1 pad 54: unconnected-(J1D-R11-Pad54) -> /R11
- J1 pad 55: unconnected-(J1D-R10-Pad55) -> /R10
- J1 pad 57: unconnected-(J1D-RCLK-Pad57) -> /RCLK
- J1 pad 59: unconnected-(J1D-R07-Pad59) -> /R07
- J1 pad 6: unconnected-(J1A-T23-Pad6) -> /T23
- J1 pad 60: unconnected-(J1D-R06-Pad60) -> /R06
- J1 pad 61: unconnected-(J1D-R05-Pad61) -> /R05
- J1 pad 62: unconnected-(J1D-R04-Pad62) -> /R04
- J1 pad 63: unconnected-(J1D-R03-Pad63) -> /R03
- J1 pad 64: unconnected-(J1D-R02-Pad64) -> /R02
- J1 pad 65: unconnected-(J1D-R01-Pad65) -> /R01
- J1 pad 66: unconnected-(J1D-R00-Pad66) -> /R00
- J1 pad 7: unconnected-(J1A-T22-Pad7) -> /T22
- J1 pad 70: unconnected-(J1C-B27-Pad70) -> /B27
- J1 pad 71: unconnected-(J1C-B26-Pad71) -> /B26
- J1 pad 72: unconnected-(J1C-B25-Pad72) -> /B25
- J1 pad 73: unconnected-(J1C-B24-Pad73) -> /B24
- J1 pad 74: unconnected-(J1C-B23-Pad74) -> /B23
- J1 pad 75: unconnected-(J1C-B22-Pad75) -> /B22
- J1 pad 76: unconnected-(J1C-B21-Pad76) -> /B21
- J1 pad 77: unconnected-(J1C-B20-Pad77) -> /B20
- J1 pad 78: GND -> /BX3
- J1 pad 79: unconnected-(J1C-BY-Pad79) -> /BX2
- J1 pad 8: unconnected-(J1A-T21-Pad8) -> /T21
- J1 pad 80: unconnected-(J1C-BX-Pad80) -> /BX1
- J1 pad 81: GND -> /BX0
- J1 pad 82: unconnected-(J1C-B17-Pad82) -> /B17
- J1 pad 83: unconnected-(J1C-B16-Pad83) -> /B16
- J1 pad 84: unconnected-(J1C-B15-Pad84) -> /B15
- J1 pad 85: unconnected-(J1C-B14-Pad85) -> /B14
- J1 pad 86: unconnected-(J1C-B13-Pad86) -> /B13
- J1 pad 87: unconnected-(J1C-B12-Pad87) -> /B12
- J1 pad 88: unconnected-(J1C-B11-Pad88) -> /B11
- J1 pad 89: unconnected-(J1C-B10-Pad89) -> /B10
- J1 pad 9: unconnected-(J1A-T20-Pad9) -> /T20
- J1 pad 91: unconnected-(J1C-BCLK-Pad91) -> /BCLK
- J1 pad 93: unconnected-(J1C-B07-Pad93) -> /B07
- J1 pad 94: unconnected-(J1C-B06-Pad94) -> /B06
- J1 pad 95: unconnected-(J1C-B05-Pad95) -> /B05
- J1 pad 96: unconnected-(J1C-B04-Pad96) -> /B04
- J1 pad 97: unconnected-(J1C-B03-Pad97) -> /B03
- J1 pad 98: unconnected-(J1C-B02-Pad98) -> /B02
- J1 pad 99: unconnected-(J1C-B01-Pad99) -> /B01
