File: hardware/v33/v33.kicad_sch (KiCad schematic)
At the start: 10 parts, among them J1 nuMezzanine_4x34, U1 uPD70136L-16

Commit message: Update mainboard to revision 2
Add an additional 8 bidirectional channels
Replace SPI PSRAM with hyperram
Remove LEDs
Parts:
- C1, C2, C3, C4: footprint Capacitor_THT:C_Disc_D5.0mm_W2.5mm_P5.00mm -> Capacitor_SMD:C_0805_2012Metric_Pad1.18x1.45mm_HandSolder
- R1, R2, R3, R4: footprint Resistor_THT:R_Axial_DIN0207_L6.3mm_D2.5mm_P7.62mm_Horizontal -> Resistor_SMD:R_0805_2012Metric_Pad1.20x1.40mm_HandSolder
Connections:
- net GND: now also J1.102 (GND), J1.136 (GND); no longer J1.10 (GND), J1.112 (GND), J1.115 (GND), J1.13 (GND), J1.44 (GND), J1.47 (GND), J1.78 (GND), J1.81 (GND)
- no-connect marks 39 -> 47
Changed lines of the file:
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@@
           (size 1.27 1.27))
         (justify left)))
-    (property "Footprint" "Capacitor_THT:C_Disc_D5.0mm_W2.5mm_P5.00mm"
+    (property "Footprint" "Capacitor_SMD:C_0805_2012Metric_Pad1.18x1.45mm_HandSolder"
       (at 218.44 116.84 0)
       (hide yes)
@@
           (size 1.27 1.27))
         (justify left)))
-    (property "Footprint" "Capacitor_THT:C_Disc_D5.0mm_W2.5mm_P5.00mm"
+    (property "Footprint" "Capacitor_SMD:C_0805_2012Metric_Pad1.18x1.45mm_HandSolder"
       (at 243.84 116.84 0)
       (hide yes)
@@
           (size 1.27 1.27))
         (justify left)))
-    (property "Footprint" "Capacitor_THT:C_Disc_D5.0mm_W2.5mm_P5.00mm"
+    (property "Footprint" "Capacitor_SMD:C_0805_2012Metric_Pad1.18x1.45mm_HandSolder"
       (at 269.24 116.84 0)
       (hide yes)
@@
           (size 1.27 1.27))
         (justify left)))
-    (property "Footprint" "Capacitor_THT:C_Disc_D5.0mm_W2.5mm_P5.00mm"
+    (property "Footprint" "Capacitor_SMD:C_0805_2012Metric_Pad1.18x1.45mm_HandSolder"
       (at 294.64 116.84 0)
       (hide yes)
@@
           (size 1.0 1.0))
         (justify left)))
-    (property "Footprint" "Resistor_THT:R_Axial_DIN0207_L6.3mm_D2.5mm_P7.62mm_Horizontal"
+    (property "Footprint" "Resistor_SMD:R_0805_2012Metric_Pad1.20x1.40mm_HandSolder"
       (at 129.54 224.79 0)
       (effects
@@
           (size 1.0 1.0))
         (justify left)))
-    (property "Footprint" "Resistor_THT:R_Axial_DIN0207_L6.3mm_D2.5mm_P7.62mm_Horizontal"
+    (property "Footprint" "Resistor_SMD:R_0805_2012Metric_Pad1.20x1.40mm_HandSolder"
       (at 170.18 224.79 0)
       (effects
@@
           (size 1.0 1.0))
         (justify left)))
-    (property "Footprint" "Resistor_THT:R_Axial_DIN0207_L6.3mm_D2.5mm_P7.62mm_Horizontal"
+    (property "Footprint" "Resistor_SMD:R_0805_2012Metric_Pad1.20x1.40mm_HandSolder"
       (at 210.82 224.79 0)
       (effects
@@
           (size 1.0 1.0))
         (justify left)))
-    (property "Footprint" "Resistor_THT:R_Axial_DIN0207_L6.3mm_D2.5mm_P7.62mm_Horizontal"
+    (property "Footprint" "Resistor_SMD:R_0805_2012Metric_Pad1.20x1.40mm_HandSolder"
       (at 251.46 224.79 0)
       (effects
@@
       (font
         (size 1.1 1.1)))
-))
+)(no_connect (at 36.83 186.69))
+(no_connect (at 36.83 194.31))
+(no_connect (at 36.83 95.25))
+(no_connect (at 36.83 102.87))
+(no_connect (at 72.39 186.69))
+(no_connect (at 72.39 194.31))
+(no_connect (at 72.39 95.25))
+(no_connect (at 72.39 102.87))
+)
