File: hardware/z80/z80.kicad_sch (KiCad schematic)
At the start: 13 parts, among them J1 nuMezzanine_4x34, U1 Z84C0008PEG

Commit message: Update mainboard to revision 2
Add an additional 8 bidirectional channels
Replace SPI PSRAM with hyperram
Remove LEDs
Parts:
- C1: footprint Capacitor_THT:C_Disc_D5.0mm_W2.5mm_P5.00mm -> Capacitor_SMD:C_0805_2012Metric_Pad1.18x1.45mm_HandSolder
- R1, R10, R11, R2, R4, R5, R6, R7, R8, R9: footprint Resistor_THT:R_Axial_DIN0207_L6.3mm_D2.5mm_P7.62mm_Horizontal -> Resistor_SMD:R_0805_2012Metric_Pad1.20x1.40mm_HandSolder
Connections:
- net GND: now also J1.102 (GND), J1.136 (GND); no longer J1.10 (GND), J1.112 (GND), J1.115 (GND), J1.13 (GND), J1.44 (GND), J1.47 (GND), J1.78 (GND), J1.81 (GND)
- net BY renamed BX2
- net LX renamed LX1
- net LY renamed LX2
- net RX renamed RX1
- no-connect marks 51 -> 59
Changed lines of the file:
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@@
       (justify left bottom))
 )
-  (label "LY"
+  (label "LX2"
     (at 36.83 191.77 0)
     (effects
@@
       (justify left bottom))
 )
-  (label "BY"
+  (label "BX2"
     (at 72.39 100.33 0)
     (effects
@@
       (justify left bottom))
 )
-  (label "RX"
+  (label "RX1"
     (at 72.39 189.23 0)
     (effects
@@
       (justify left bottom))
 )
-  (label "LX"
+  (label "LX1"
     (at 36.83 189.23 0)
     (effects
@@
       (type default))
 )
-  (label "LX"
+  (label "LX1"
     (at 160.02 114.3 180)
     (effects
@@
       (type default))
 )
-  (label "LY"
+  (label "LX2"
     (at 160.02 116.84 180)
     (effects
@@
       (type default))
 )
-  (label "BY"
+  (label "BX2"
     (at 160.02 104.14 180)
     (effects
@@
       (type default))
 )
-  (label "RX"
+  (label "RX1"
     (at 160.02 129.54 180)
     (effects
@@
         (font
           (size 1.27 1.27))))
-    (property "Footprint" "Capacitor_THT:C_Disc_D5.0mm_W2.5mm_P5.00mm"
+    (property "Footprint" "Capacitor_SMD:C_0805_2012Metric_Pad1.18x1.45mm_HandSolder"
       (at 233.68 78.74 0)
       (hide yes)
@@
         (font
           (size 1.27 1.27))))
-    (property "Footprint" "Resistor_THT:R_Axial_DIN0207_L6.3mm_D2.5mm_P7.62mm_Horizontal"
+    (property "Footprint" "Resistor_SMD:R_0805_2012Metric_Pad1.20x1.40mm_HandSolder"
       (at 215.9 116.84 0)
       (hide yes)
@@
       (type default))
 )
-  (label "LX"
+  (label "LX1"
     (at 215.9 124.46 0)
     (effects
@@
         (font
           (size 1.27 1.27))))
-    (property "Footprint" "Resistor_THT:R_Axial_DIN0207_L6.3mm_D2.5mm_P7.62mm_Horizontal"
+    (property "Footprint" "Resistor_SMD:R_0805_2012Metric_Pad1.20x1.40mm_HandSolder"
       (at 228.6 116.84 0)
       (hide yes)
@@
       (type default))
 )
-  (label "LY"
+  (label "LX2"
     (at 228.6 124.46 0)
     (effects
@@
         (font
           (size 1.27 1.27))))
-    (property "Footprint" "Resistor_THT:R_Axial_DIN0207_L6.3mm_D2.5mm_P7.62mm_Horizontal"
+    (property "Footprint" "Resistor_SMD:R_0805_2012Metric_Pad1.20x1.40mm_HandSolder"
       (at 254.0 116.84 0)
       (hide yes)
@@
       (type default))
 )
-  (label "BY"
+  (label "BX2"
     (at 254.0 124.46 0)
     (effects
@@
         (font
           (size 1.27 1.27))))
-    (property "Footprint" "Resistor_THT:R_Axial_DIN0207_L6.3mm_D2.5mm_P7.62mm_Horizontal"
+    (property "Footprint" "Resistor_SMD:R_0805_2012Metric_Pad1.20x1.40mm_HandSolder"
       (at 266.7 116.84 0)
       (hide yes)
@@
       (type default))
 )
-  (label "RX"
+  (label "RX1"
     (at 266.7 124.46 0)
     (effects
@@
           (size 1.0 1.0))
         (justify left)))
-    (property "Footprint" "Resistor_THT:R_Axial_DIN0207_L6.3mm_D2.5mm_P7.62mm_Horizontal"
+    (property "Footprint" "Resistor_SMD:R_0805_2012Metric_Pad1.20x1.40mm_HandSolder"
       (at 129.54 224.79 0)
       (effects
@@
           (size 1.0 1.0))
         (justify left)))
-    (property "Footprint" "Resistor_THT:R_Axial_DIN0207_L6.3mm_D2.5mm_P7.62mm_Horizontal"
+    (property "Footprint" "Resistor_SMD:R_0805_2012Metric_Pad1.20x1.40mm_HandSolder"
       (at 170.18 224.79 0)
       (effects
@@
           (size 1.0 1.0))
         (justify left)))
-    (property "Footprint" "Resistor_THT:R_Axial_DIN0207_L6.3mm_D2.5mm_P7.62mm_Horizontal"
+    (property "Footprint" "Resistor_SMD:R_0805_2012Metric_Pad1.20x1.40mm_HandSolder"
       (at 210.82 224.79 0)
       (effects
@@
           (size 1.0 1.0))
         (justify left)))
-    (property "Footprint" "Resistor_THT:R_Axial_DIN0207_L6.3mm_D2.5mm_P7.62mm_Horizontal"
+    (property "Footprint" "Resistor_SMD:R_0805_2012Metric_Pad1.20x1.40mm_HandSolder"
       (at 251.46 224.79 0)
       (effects
@@
           (size 1.0 1.0))
         (justify left)))
-    (property "Footprint" "Resistor_THT:R_Axial_DIN0207_L6.3mm_D2.5mm_P7.62mm_Horizontal"
+    (property "Footprint" "Resistor_SMD:R_0805_2012Metric_Pad1.20x1.40mm_HandSolder"
       (at 292.1 224.79 0)
       (effects
@@
           (size 1.0 1.0))
         (justify left)))
-    (property "Footprint" "Resistor_THT:R_Axial_DIN0207_L6.3mm_D2.5mm_P7.62mm_Horizontal"
+    (property "Footprint" "Resistor_SMD:R_0805_2012Metric_Pad1.20x1.40mm_HandSolder"
       (at 332.74 224.79 0)
       (effects
@@
       (font
         (size 1.1 1.1)))
-))
+)(no_connect (at 36.83 186.69))
+(no_connect (at 36.83 194.31))
+(no_connect (at 36.83 95.25))
+(no_connect (at 36.83 102.87))
+(no_connect (at 72.39 186.69))
+(no_connect (at 72.39 194.31))
+(no_connect (at 72.39 95.25))
+(no_connect (at 72.39 102.87))
+)
